Commit message: t2 working skid steer drive

File: src/t2/urdf/b2.xacro (robot description, xacro)
@@ -1,4 +1,5 @@
 <?xml version="1.0" ?>
-<robot name="m2wr" xmlns:xacro="http://www.ros.org/wiki/xacro">
+<robot name="skid_steer_bot" xmlns:xacro="http://www.ros.org/wiki/xacro">
+  <!-- Colors
   <material name="black">
     <color rgba="0.0 0.0 0.0 1.0"/>
@@ -25,4 +26,5 @@
     <color rgba="1.0 1.0 1.0 1.0"/>
   </material>
+  -->
   <gazebo reference="link_chassis">
     <material>Gazebo/Orange</material>
@@ -35,19 +37,40 @@
   </gazebo>
   <gazebo>
-    <plugin filename="libgazebo_ros_diff_drive.so" name="differential_drive_controller">
-      <legacyMode>false</legacyMode>
-      <alwaysOn>true</alwaysOn>
-      <updateRate>20</updateRate>
-      <leftJoint>joint_left_wheel</leftJoint>
-      <rightJoint>joint_right_wheel</rightJoint>
-      <wheelSeparation>0.2</wheelSeparation>
+      <plugin name="skid_steer_drive_controller" filename="libgazebo_ros_skid_steer_drive.so">
+      <updateRate>100.0</updateRate>
+      <robotNamespace>/</robotNamespace>
+      <leftFrontJoint>front_left_wheel_joint</leftFrontJoint>
+      <rightFrontJoint>front_right_wheel_joint</rightFrontJoint>
+      <leftRearJoint>back_left_wheel_joint</leftRearJoint>
+      <rightRearJoint>back_right_wheel_joint</rightRearJoint>
+      <wheelSeparation>0.3</wheelSeparation>
       <wheelDiameter>0.2</wheelDiameter>
-      <torque>0.1</torque>
-      <commandTopic>cmd_vel</commandTopic>
-      <odometryTopic>odom</odometryTopic>
-      <odometryFrame>odom</odometryFrame>
-      <robotBaseFrame>link_chassis</robotBaseFrame>
+      <robotBaseFrame>base_link</robotBaseFrame>
+      <torque>20</torque>
+      <topicName>cmd_vel</topicName>
+      <broadcastTF>false</broadcastTF>
     </plugin>
   </gazebo>
+  <xacro:property name="wheel_radius" value="0.2"/>
+  <xacro:macro name="wheel_inertial">
+    <inertial>
+      <mass value="0.2"/>
+      <origin rpy="0 1.5707 1.5707" xyz="0 0 0"/>
+      <inertia ixx="0.000526666666667" ixy="0" ixz="0" iyy="0.000526666666667"
+        iyz="0" izz="0.001"/>
+    </inertial>
+  </xacro:macro>
+  <xacro:macro name="wheel_collision_values">
+    <origin rpy="0 1.5707 1.5707" xyz="0 0 0"/>
+    <geometry>
+      <cylinder length="0.04" radius="0.1"/>
+    </geometry>
+  </xacro:macro>
+  <xacro:macro name="wheel_visual_values">
+    <origin rpy="0 1.5707 1.5707" xyz="0 0 0"/>
+    <geometry>
+      <cylinder length="0.04" radius="0.1"/>
+    </geometry>
+  </xacro:macro>
   <link name="link_chassis">
     <!-- pose and inertial -->
@@ -72,85 +95,114 @@
       <material name="blue"/>
     </visual>
-    <!-- caster front -->
-    <collision name="caster_front_collision">
-      <origin rpy=" 0 0 0" xyz="0.2 0 -0.05"/>
-      <geometry>
-        <sphere radius="0.05"/>
-      </geometry>
-      <surface>
-        <friction>
-          <ode>
-            <mu>0.00001</mu>
-            <mu2>0.00001</mu2>
-            <slip1>1.0</slip1>
-            <slip2>1.0</slip2>
-          </ode>
-        </friction>
-      </surface>
-    </collision>
-    <visual name="caster_front_visual">
-      <origin rpy=" 0 0 0" xyz="0.2 0 -0.05"/>
-      <geometry>
-        <sphere radius="0.05"/>
-      </geometry>
-    </visual>
-    <inertial>
-      <mass value="100"/>
-      <origin rpy="0 0 0" xyz="0.2 0 -0.05"/>
-      <inertia ixx="0.1" ixy="0" ixz="0" iyy="0.1"
-        iyz="0" izz="0.1"/>
-    </inertial>
-  </link>
-  <link name="link_right_wheel">
-    <inertial>
-      <mass value="0.2"/>
-      <origin rpy="0 1.5707 1.5707" xyz="0 0 0"/>
-      <inertia ixx="0.000526666666667" ixy="0" ixz="0" iyy="0.000526666666667"
-        iyz="0" izz="0.001"/>
-    </inertial>
-    <collision name="link_right_wheel_collision">
-      <origin rpy="0 1.5707 1.5707" xyz="0 0 0"/>
-      <geometry>
-        <cylinder length="0.04" radius="0.1"/>
-      </geometry>
-    </collision>
-    <visual name="link_right_wheel_visual">
-      <origin rpy="0 1.5707 1.5707" xyz="0 0 0"/>
-      <geometry>
-        <cylinder length="0.04" radius="0.1"/>
-      </geometry>
-    </visual>
-  </link>
-  <joint name="joint_right_wheel" type="continuous">
-    <origin rpy="0 0 0" xyz="-0.05 0.15 0"/>
-    <child link="link_right_wheel"/>
-    <parent link="link_chassis"/>
-    <axis rpy="0 0 0" xyz="0 1 0"/>
-    <limit effort="100" velocity="1"/>
-    <joint_properties damping="1.0" friction="1.0"/>
-  </joint>
-  <link name="link_left_wheel">
-    <inertial>
-      <mass value="0.2"/>
-      <origin rpy="0 1.5707 1.5707" xyz="0 0 0"/>
-      <inertia ixx="0.000526666666667" ixy="0" ixz="0" iyy="0.000526666666667"
-        iyz="0" izz="0.001"/>
-    </inertial>
-    <collision name="link_left_wheel_collision">
-      <origin rpy="0 1.5707 1.5707" xyz="0 0 0"/>
-      <geometry>
-        <cylinder length="0.04" radius="0.1"/>
-      </geometry>
-    </collision>
-    <visual name="link_left_wheel_visual">
-      <origin rpy="0 1.5707 1.5707" xyz="0 0 0"/>
-      <geometry>
-        <cylinder length="0.04" radius="0.1"/>
-      </geometry>
-    </visual>
-  </link>
-  <joint name="joint_left_wheel" type="continuous">
-    <origin rpy="0 0 0" xyz="-0.05 -0.15 0"/>
-    <child link="link_left_wheel"/>
+  </link>
+  <!-- defining wheels -->
+  <link name="link_front_right_wheel">
+    <inertial>
+      <mass value="0.2"/>
+      <origin rpy="0 1.5707 1.5707" xyz="0 0 0"/>
+      <inertia ixx="0.000526666666667" ixy="0" ixz="0" iyy="0.000526666666667"
+        iyz="0" izz="0.001"/>
+    </inertial>
+    <collision name="link_front_right_wheel_collision">
+      <origin rpy="0 1.5707 1.5707" xyz="0 0 0"/>
+    <geometry>
+      <cylinder length="0.04" radius="0.1"/>
+    </geometry>
+    </collision>
+    <visual name="link_front_right_wheel_visual">
+      <origin rpy="0 1.5707 1.5707" xyz="0 0 0"/>
+    <geometry>
+      <cylinder length="0.04" radius="0.1"/>
+    </geometry>
+    </visual>
+  </link>
+  <link name="link_front_left_wheel">
+    <inertial>
+      <mass value="0.2"/>
+      <origin rpy="0 1.5707 1.5707" xyz="0 0 0"/>
+      <inertia ixx="0.000526666666667" ixy="0" ixz="0" iyy="0.000526666666667"
+        iyz="0" izz="0.001"/>
+    </inertial>
+    <collision name="link_front_left_wheel_collision">
+      <origin rpy="0 1.5707 1.5707" xyz="0 0 0"/>
+    <geometry>
+      <cylinder length="0.04" radius="0.1"/>
+    </geometry>
+    </collision>
+    <visual name="link_front_left_wheel_visual">
+      <origin rpy="0 1.5707 1.5707" xyz="0 0 0"/>
+    <geometry>
+      <cylinder length="0.04" radius="0.1"/>
+    </geometry>
+    </visual>
+  </link>
+  <link name="link_back_right_wheel">
+    <inertial>
+      <mass value="0.2"/>
+      <origin rpy="0 1.5707 1.5707" xyz="0 0 0"/>
+      <inertia ixx="0.000526666666667" ixy="0" ixz="0" iyy="0.000526666666667"
+        iyz="0" izz="0.001"/>
+    </inertial>
+    <collision name="link_back_right_wheel_collision">
+      <origin rpy="0 1.5707 1.5707" xyz="0 0 0"/>
+    <geometry>
+      <cylinder length="0.04" radius="0.1"/>
+    </geometry>
+    </collision>
+    <visual name="link_back_right_wheel_visual">
+      <origin rpy="0 1.5707 1.5707" xyz="0 0 0"/>
+    <geometry>
+      <cylinder length="0.04" radius="0.1"/>
+    </geometry>
+    </visual>
+  </link>
+  <link name="link_back_left_wheel">
+    <inertial>
+      <mass value="0.2"/>
+      <origin rpy="0 1.5707 1.5707" xyz="0 0 0"/>
+      <inertia ixx="0.000526666666667" ixy="0" ixz="0" iyy="0.000526666666667"
+        iyz="0" izz="0.001"/>
+    </inertial>
+    <collision name="link_back_left_wheel_collision">
+      <origin rpy="0 1.5707 1.5707" xyz="0 0 0"/>
+    <geometry>
+      <cylinder length="0.04" radius="0.1"/>
+    </geometry>
+    </collision>
+    <visual name="link_back_left_wheel_visual">
+      <origin rpy="0 1.5707 1.5707" xyz="0 0 0"/>
+    <geometry>
+      <cylinder length="0.04" radius="0.1"/>
+    </geometry>
+    </visual>
+  </link>
+  <!-- defining joints -->
+  <joint name="front_right_wheel_joint" type="continuous">
+    <origin rpy="0 0 0" xyz="0.15 0.15 0"/>
+    <child link="link_front_right_wheel"/>
+    <parent link="link_chassis"/>
+    <axis rpy="0 0 0" xyz="0 1 0"/>
+    <limit effort="100" velocity="1"/>
+    <joint_properties damping="1.0" friction="1.0"/>
+  </joint>
+  <joint name="front_left_wheel_joint" type="continuous">
+    <origin rpy="0 0 0" xyz="0.15 -0.15 0"/>
+    <child link="link_front_left_wheel"/>
+    <parent link="link_chassis"/>
+    <axis rpy="0 0 0" xyz="0 1 0"/>
+    <limit effort="100" velocity="1"/>
+    <joint_properties damping="1.0" friction="1.0"/>
+  </joint>
+  <joint name="back_right_wheel_joint" type="continuous">
+    <origin rpy="0 0 0" xyz="-0.15 0.15 0"/>
+    <child link="link_back_right_wheel"/>
+    <parent link="link_chassis"/>
+    <axis rpy="0 0 0" xyz="0 1 0"/>
+    <limit effort="100" velocity="1"/>
+    <joint_properties damping="1.0" friction="1.0"/>
+  </joint>
+  <joint name="back_left_wheel_joint" type="continuous">
+    <origin rpy="0 0 0" xyz="-0.15 -0.15 0"/>
+    <child link="link_back_left_wheel"/>
     <parent link="link_chassis"/>
     <axis rpy="0 0 0" xyz="0 1 0"/>
